Commit message: display update

File: src/Hanuman/urdf/hanuman.xacro (robot description, xacro)
@@ -148,4 +148,9 @@
     <xacro:macro name="humanoid" params="parent">
         <xacro:robot_link link_name="torso" collision_enable="true"/>
+        <joint name="torso_to_world" type="fixed">
+            <parent link="${parent}"/>
+            <child link="torso"/>
+            <origin xyz="0 0 0.9" rpy="0 0 0"/>
+        </joint>
         <!-- <xacro:head_assem/>
         <xacro:L_arm_assem/>
